File: Amplificador_Push_Pull_AB/Amplificador_Push_Pull_AB.brd (EAGLE design)
At the start: 99 x 49.8 mm, 51 parts, among them IC1 LM741P, P2 10k, Q1 BC547, Q10 TIP42C, Q2 BC547, Q4 BC547, Q7 BC547, Q8 BC547, T2 2SC1307

Commit message: One connection left.
Parts:
- removed IC2: (no value), SparkFun-PowerIC:TO-220-ALT
- added IC3: 788TV, linear:TO220V
- R3: value (none) -> 13k
- moved C5 98.4 mm to (41.9, 41.9), turned to 90 degrees
- moved RLEFT 82.0 mm to (76.8, 8.26), turned to 90 degrees
- moved RIN 81.3 mm to (57.1, 10.8), turned to 90 degrees
- moved RIN2 80.0 mm to (49.5, 12.1), turned to 180 degrees
- moved C6 77.6 mm to (49.5, 40.0), turned to 270 degrees
- moved RIN1 67.0 mm to (71.1, 12.1), flipped to the bottom, turned to 90 degrees
- moved IC1 63.1 mm to (64.1, 10.8), turned to 180 degrees
- moved RMIC 60.2 mm to (84.5, 25.4), turned to 180 degrees
- moved C7 57.7 mm to (83.2, 29.8), turned to 180 degrees
- moved C8 55.6 mm to (77.5, 29.8), turned to 180 degrees
- moved C2 42.6 mm to (10.8, 19.1), turned to 270 degrees
- moved Q11 37.3 mm to (83.2, 19.1), turned to 270 degrees
- moved C1 13.1 mm to (78.7, 41.9)
- moved Q10 6.63 mm to (55.9, 22.9)
- moved REC1 5.12 mm to (70.5, 33.7)
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Connections:
- removed net N$18: RLEFT.2
- net +18V: now also IC3.1; no longer IC2.IN
- net GND: now also IC3.2; no longer IC2.GND
- net N$20: now also RLEFT.2
- net N$24: now also IC3.3; no longer IC2.OUT
Routing:
- net GND: track 93.0 -> 220.7 mm, vias 4 -> 12
- net N$30: track 0.00 -> 100.5 mm, vias 0 -> 2
- net N$20: track 0.00 -> 73.4 mm, vias 0 -> 2
- net VOUT: track 0.00 -> 52.3 mm, vias 0 -> 2
- net -18V: track 125.9 -> 174.0 mm, vias 0 -> 2
- net N$25: track 0.00 -> 39.8 mm
- net +18V: track 120.4 -> 159.8 mm, vias 2 -> 4
- net N$19: track 6.35 -> 31.9 mm
- net N$26: track 0.00 -> 23.7 mm
- net N$14: track 0.00 -> 16.3 mm
- net N$24: track 0.00 -> 15.3 mm
- net N$9: track 0.00 -> 15.0 mm
- net N$27: track 0.00 -> 10.9 mm
- net N$12: track 0.00 -> 9.04 mm
- net N$21: track 0.00 -> 8.15 mm
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
Commit message: Board finished. Need to verify.
Parts:
- RIN1, RLEFT, RRIGHT: device rcl:0207/10 -> rcl:0207/7
- moved P1 3.42 mm to (19.7, 13.3)
- moved REB2 3.42 mm to (31.1, 13.3)
- moved Q9 3.42 mm to (45.7, 21.0)
- moved RIN2 3.24 mm to (46.4, 12.7)
- moved RBC 2.69 mm to (45.7, 29.2)
- moved JP2 2.54 mm to (11.4, 7.62)
- moved C2 1.90 mm to (10.8, 21.0)
- moved RLEFT 1.80 mm to (78.1, 6.99)
- moved RRIGHT 1.80 mm to (75.6, 6.99)
- moved RIN1 1.80 mm to (72.4, 10.8)
- moved C5 1.42 mm to (41.3, 43.2)
- moved RMIC 1.42 mm to (85.7, 26.0)
- moved C6 1.42 mm to (48.9, 41.3)
- moved C3 1.27 mm to (48.9, 35.6), turned to 0 degrees
- moved IC1 1.27 mm to (62.9, 10.8)
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Routing:
- net N$27: track 10.9 -> 64.8 mm, vias 0 -> 4
- net GND: track 220.7 -> 272.5 mm
- net N$16: track 17.0 -> 9.94 mm
- net VOUT: track 52.3 -> 57.4 mm
- net N$26: track 23.7 -> 28.6 mm
- net N$25: track 39.8 -> 44.0 mm
- net N$17: track 26.7 -> 23.1 mm
- net -18V: track 174.0 -> 177.1 mm
- net N$30: track 100.5 -> 103.5 mm
- net +18V: track 159.8 -> 162.5 mm
- net P1: track 59.1 -> 61.7 mm
- net N$15: track 26.5 -> 28.6 mm
- net N$22: track 3.44 -> 4.97 mm
- net VIN: track 8.52 -> 7.25 mm
- net N$20: track 73.4 -> 74.6 mm
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