File: Amplificador_Push_Pull_AB/Amplificador_Push_Pull_AB.sch (EAGLE design)
At the start: 51 parts, among them IC1 LM741P, P2 10k, Q1 BC547, Q10 TIP42C, Q2 BC547, Q4 BC547, Q7 BC547, Q8 BC547, T2 2SC1307

Commit message: One connection left.
Parts:
- removed IC2: (no value), SparkFun-PowerIC:V_REG_78XX-TO-220
- added IC3: 788TV, linear:788TV
- R3: value (none) -> 13k
Connections:
- removed net N$18: RLEFT.2
- net +18V: now also IC3.VI; no longer IC2.IN
- net GND: now also IC3.GND; no longer IC2.GND
- net N$20: now also RLEFT.2
- net N$24: now also IC3.VO; no longer IC2.OUT

Commit message: Board finished. Need to verify.
Parts:
- RIN1, RLEFT, RRIGHT: device rcl:R-EU_0207/10 -> rcl:R-EU_0207/7
Changed lines of the file:
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@@
 <part name="JP1" library="SparkFun-Connectors" deviceset="AUDIO-JACK" device="PTH"/>
 <part name="GND8" library="supply1" deviceset="GND" device=""/>
-<part name="RRIGHT" library="rcl" deviceset="R-EU_" device="0207/10" value="10k"/>
+<part name="RRIGHT" library="rcl" deviceset="R-EU_" device="0207/7" value="10k"/>
 <part name="RMIC" library="rcl" deviceset="R-EU_" device="0207/10" value="10k"/>
 <part name="GND9" library="supply1" deviceset="GND" device=""/>
@@
 <part name="RIN" library="rcl" deviceset="R-EU_" device="0207/10" value="100k"/>
 <part name="GND12" library="supply1" deviceset="GND" device=""/>
-<part name="RIN1" library="rcl" deviceset="R-EU_" device="0207/10" value="100k"/>
+<part name="RIN1" library="rcl" deviceset="R-EU_" device="0207/7" value="100k"/>
 <part name="RIN2" library="rcl" deviceset="R-EU_" device="0207/10" value="10k"/>
 <part name="GND13" library="supply1" deviceset="GND" device=""/>
@@
 <part name="JP2" library="pinhead" deviceset="PINHD-1X3" device=""/>
 <part name="GND14" library="supply1" deviceset="GND" device=""/>
-<part name="RLEFT" library="rcl" deviceset="R-EU_" device="0207/10" value="10k"/>
+<part name="RLEFT" library="rcl" deviceset="R-EU_" device="0207/7" value="10k"/>
 <part name="IC3" library="linear" deviceset="78*" device="TV" technology="8"/>
 </parts>
